Commit message: fixed urdf

File: ros_basics_exercise/urdf/thymio_simple.urdf (robot description, URDF)
Before this commit: robot thymio, 4 links, 3 joints
Links:
- removed link castor_link
- added link sensor_back_left, mass 0.001; collision box size=0.007 0.0025 0.004; visual box size=0.007 0.0025 0.004
- added link sensor_back_right, mass 0.001; collision box size=0.007 0.0025 0.004; visual box size=0.007 0.0025 0.004
- added link sensor_center, mass 0.001; collision box size=0.007 0.0025 0.004; visual box size=0.007 0.0025 0.004
- added link sensor_center_left, mass 0.001; collision box size=0.007 0.0025 0.004; visual box size=0.007 0.0025 0.004
- added link sensor_center_right, mass 0.001; collision box size=0.007 0.0025 0.004; visual box size=0.007 0.0025 0.004
- added link sensor_left, mass 0.001; collision box size=0.007 0.0025 0.004; visual box size=0.007 0.0025 0.004
- added link sensor_right, mass 0.001; collision box size=0.007 0.0025 0.004; visual box size=0.007 0.0025 0.004
- link base_link: geometry collision box size=0.11 0.112 0.045; collision sphere radius=0.01
Joints:
- removed joint castor_joint
- added joint base_link_sensor_back_left: type fixed, parent base_link, child sensor_back_left, origin xyz=0 0 0 rpy=0 0 0
- added joint base_link_sensor_back_right: type fixed, parent base_link, child sensor_back_right, origin xyz=0 0 0 rpy=0 0 0
- added joint base_link_sensor_center: type fixed, parent base_link, child sensor_center, origin xyz=0 0 0 rpy=0 0 0
- added joint base_link_sensor_center_left: type fixed, parent base_link, child sensor_center_left, origin xyz=0 0 0 rpy=0 0 0
- added joint base_link_sensor_center_right: type fixed, parent base_link, child sensor_center_right, origin xyz=0 0 0 rpy=0 0 0
- added joint base_link_sensor_left: type fixed, parent base_link, child sensor_left, origin xyz=0 0 0 rpy=0 0 0
- added joint base_link_sensor_right: type fixed, parent base_link, child sensor_right, origin xyz=0 0 0 rpy=0 0 0
- joint left_wheel_joint: origin xyz=-0.02 0.049 -0.007 rpy=0 0 0 -> xyz=-0.024 0.049 -0.007 rpy=0 0 0
- joint right_wheel_joint: origin xyz=-0.02 -0.049 -0.007 rpy=0 0 0 -> xyz=-0.024 -0.049 -0.007 rpy=0 0 0

File: ros_basics_exercise/urdf/thymio_simple.urdf.xacro (robot description, xacro)
@@ -106,10 +106,10 @@
     </joint>
     <!-- Add your sensors using the macro -->
-    <xacro:csensor plink="base_link" id="sensor_center" mass="0.001" originrpy="0 0 1.5708" originxyz="0.066 0 0" jointxyz="0 0 0" jointrpy="0 0 0" />
-    <xacro:csensor plink="base_link" id="sensor_center_right" mass="0.001" originrpy="0 0 1.309" originxyz="0.064 -0.0275 0" jointxyz="0 0 0" jointrpy="0 0 0" />
-    <xacro:csensor plink="base_link" id="sensor_center_left" mass="0.001" originrpy="0 0 1.8326" originxyz="0.064 0.0275 0" jointxyz="0 0 0" jointrpy="0 0 0" />
-    <xacro:csensor plink="base_link" id="sensor_right" mass="0.001" originrpy="0 0 1.0472" originxyz="0.058 -0.055 0" jointxyz="0 0 0" jointrpy="0 0 0" />
-    <xacro:csensor plink="base_link" id="sensor_left" mass="0.001" originrpy="0 0 2.26893" originxyz="0.058 0.055 0" jointxyz="0 0 0" jointrpy="0 0 0" />
-    <xacro:csensor plink="base_link" id="sensor_back_right" mass="0.001" originrpy="0 0 1.5708" originxyz="-0.056 -0.035 0" jointxyz="0 0 0" jointrpy="0 0 0" />
-    <xacro:csensor plink="base_link" id="sensor_bacK_left" mass="0.001" originrpy="0 0 1.5708" originxyz="-0.056 0.035 0" jointxyz="0 0 0" jointrpy="0 0 0" />
+    <xacro:csensor plink="base_link" id="center" mass="0.001" originrpy="0 0 1.5708" originxyz="0.066 0 0" jointxyz="0 0 0" jointrpy="0 0 0" />
+    <xacro:csensor plink="base_link" id="center_right" mass="0.001" originrpy="0 0 1.309" originxyz="0.064 -0.0275 0" jointxyz="0 0 0" jointrpy="0 0 0" />
+    <xacro:csensor plink="base_link" id="center_left" mass="0.001" originrpy="0 0 1.8326" originxyz="0.064 0.0275 0" jointxyz="0 0 0" jointrpy="0 0 0" />
+    <xacro:csensor plink="base_link" id="right" mass="0.001" originrpy="0 0 1.0472" originxyz="0.058 -0.055 0" jointxyz="0 0 0" jointrpy="0 0 0" />
+    <xacro:csensor plink="base_link" id="left" mass="0.001" originrpy="0 0 2.26893" originxyz="0.058 0.055 0" jointxyz="0 0 0" jointrpy="0 0 0" />
+    <xacro:csensor plink="base_link" id="back_right" mass="0.001" originrpy="0 0 1.5708" originxyz="-0.056 -0.035 0" jointxyz="0 0 0" jointrpy="0 0 0" />
+    <xacro:csensor plink="base_link" id="back_left" mass="0.001" originrpy="0 0 1.5708" originxyz="-0.056 0.035 0" jointxyz="0 0 0" jointrpy="0 0 0" />
 </robot>

Commit message: add laser scan

File: ros_basics_exercise/urdf/thymio_simple.urdf (robot description, URDF)
Before this commit: robot thymio, 10 links, 9 joints
Joints:
- joint base_link_sensor_back_left: origin xyz=0 0 0 rpy=0 0 0 -> xyz=-0.056 0.035 0 rpy=0 0 0
- joint base_link_sensor_back_right: origin xyz=0 0 0 rpy=0 0 0 -> xyz=-0.056 -0.035 0 rpy=0 0 0
- joint base_link_sensor_center: origin xyz=0 0 0 rpy=0 0 0 -> xyz=0.066 0 0 rpy=0 0 0
- joint base_link_sensor_center_left: origin xyz=0 0 0 rpy=0 0 0 -> xyz=0.064 0.0275 0 rpy=0 0 0
- joint base_link_sensor_center_right: origin xyz=0 0 0 rpy=0 0 0 -> xyz=0.064 -0.0275 0 rpy=0 0 0
- joint base_link_sensor_left: origin xyz=0 0 0 rpy=0 0 0 -> xyz=0.058 0.055 0 rpy=0 0 0
- joint base_link_sensor_right: origin xyz=0 0 0 rpy=0 0 0 -> xyz=0.058 -0.055 0 rpy=0 0 0

File: ros_basics_exercise/urdf/thymio_simple.urdf.xacro (robot description, xacro)
@@ -106,5 +106,5 @@
     </joint>
     <!-- Add your sensors using the macro -->
-    <xacro:csensor plink="base_link" id="center" mass="0.001" originrpy="0 0 1.5708" originxyz="0.066 0 0" jointxyz="0 0 0" jointrpy="0 0 0" />
+    <!--<xacro:csensor plink="base_link" id="center" mass="0.001" originrpy="0 0 1.5708" originxyz="0.066 0 0" jointxyz="0 0 0" jointrpy="0 0 0" />
     <xacro:csensor plink="base_link" id="center_right" mass="0.001" originrpy="0 0 1.309" originxyz="0.064 -0.0275 0" jointxyz="0 0 0" jointrpy="0 0 0" />
     <xacro:csensor plink="base_link" id="center_left" mass="0.001" originrpy="0 0 1.8326" originxyz="0.064 0.0275 0" jointxyz="0 0 0" jointrpy="0 0 0" />
@@ -112,4 +112,11 @@
     <xacro:csensor plink="base_link" id="left" mass="0.001" originrpy="0 0 2.26893" originxyz="0.058 0.055 0" jointxyz="0 0 0" jointrpy="0 0 0" />
     <xacro:csensor plink="base_link" id="back_right" mass="0.001" originrpy="0 0 1.5708" originxyz="-0.056 -0.035 0" jointxyz="0 0 0" jointrpy="0 0 0" />
-    <xacro:csensor plink="base_link" id="back_left" mass="0.001" originrpy="0 0 1.5708" originxyz="-0.056 0.035 0" jointxyz="0 0 0" jointrpy="0 0 0" />
+    <xacro:csensor plink="base_link" id="back_left" mass="0.001" originrpy="0 0 1.5708" originxyz="-0.056 0.035 0" jointxyz="0 0 0" jointrpy="0 0 0" />-->
+    <xacro:csensor plink="base_link" id="center" mass="0.001" originrpy="0 0 1.5708" originxyz="0 0 0" jointxyz="0.066 0 0" jointrpy="0 0 0" />
+    <xacro:csensor plink="base_link" id="center_right" mass="0.001" originrpy="0 0 1.309" originxyz="0 0 0" jointxyz="0.064 -0.0275 0" jointrpy="0 0 0" />
+    <xacro:csensor plink="base_link" id="center_left" mass="0.001" originrpy="0 0 1.8326" originxyz="0 0 0" jointxyz="0.064 0.0275 0" jointrpy="0 0 0" />
+    <xacro:csensor plink="base_link" id="right" mass="0.001" originrpy="0 0 1.0472" originxyz="0 0 0" jointxyz="0.058 -0.055 0" jointrpy="0 0 0" />
+    <xacro:csensor plink="base_link" id="left" mass="0.001" originrpy="0 0 2.26893" originxyz="0 0 0" jointxyz="0.058 0.055 0" jointrpy="0 0 0" />
+    <xacro:csensor plink="base_link" id="back_right" mass="0.001" originrpy="0 0 1.5708" originxyz="0 0 0" jointxyz="-0.056 -0.035 0" jointrpy="0 0 0" />
+    <xacro:csensor plink="base_link" id="back_left" mass="0.001" originrpy="0 0 1.5708" originxyz="0 0 0" jointxyz="-0.056 0.035 0" jointrpy="0 0 0" />
 </robot>
