Commit message: lab session2

File: ros_basics_models/urdf/setup.urdf.xacro (robot description, xacro)
@@ -215,5 +215,5 @@
     </link>
     <gazebo reference="setup">
-        <material>Gazebo/WoodFloor</material>
+        <material>Gazebo/Black</material>
     </gazebo>
     <gazebo reference="stickers">
