Commit message: simulated obs avoidance works

File: ros_basics_models/urdf/box.urdf.xacro (robot description, xacro)
@@ -19,5 +19,5 @@
             <origin xyz="0 0 0"/>
             <geometry>
-                <box size="0.05 0.045 0.07"/>
+                <box size="0.023 0.045 0.08"/>
             </geometry>
             <material name="white"/>
@@ -26,5 +26,5 @@
             <origin xyz="0 0 0"/>
             <geometry>
-                <box size="0.05 0.045 0.07"/>
+                <box size="0.023 0.045 0.08"/>
             </geometry>
             <material name="white"/>
@@ -32,5 +32,5 @@
         <inertial>
             <mass value="${body_mass}"/>
-            <xacro:box_inertia mass="${body_mass}" x="0.05" y="0.045" z='0.07' />
+            <xacro:box_inertia mass="${body_mass}" x="0.023" y="0.045" z='0.08' />
         </inertial>
     </link>

File: ros_basics_models/urdf/setup.urdf.xacro (robot description, xacro)
@@ -215,5 +215,5 @@
     </link>
     <gazebo reference="setup">
-        <material>Gazebo/Black</material>
+        <material>Gazebo/WoodFloor</material>
     </gazebo>
     <gazebo reference="stickers">

File: ros_basics_p06/ros_basics_exercise/urdf/thymio_simple.urdf.xacro (robot description, xacro)
@@ -109,14 +109,14 @@
     <xacro:csensor plink="base_link" id="0" mass="0.001" originrpy="0 0 2.26893" originxyz="-0.003 0 0" jointxyz="0.058 0.055 0" jointrpy="0 0 0" />
     <!-- CL -->
-    <xacro:csensor plink="base_link" id="1" mass="0.001" originrpy="0 0 1.8326" originxyz="-0.003 0 0" jointxyz="0.067 0.0275 0" jointrpy="0 0 0" />
+    <xacro:csensor plink="base_link" id="1" mass="0.001" originrpy="0 0 1.8326" originxyz="-0.003 0 0" jointxyz="0.064 0.0275 0" jointrpy="0 0 0" />
     <!-- C -->
-    <xacro:csensor plink="base_link" id="2" mass="0.001" originrpy="0 0 1.5708" originxyz="-0.003 0 0" jointxyz="0.07 0 0" jointrpy="0 0 0" />
+    <xacro:csensor plink="base_link" id="2" mass="0.001" originrpy="0 0 1.5708" originxyz="-0.003 0 0" jointxyz="0.066 0 0" jointrpy="0 0 0" />
     <!-- CR -->
-    <xacro:csensor plink="base_link" id="3" mass="0.001" originrpy="0 0 1.309" originxyz="-0.003 0 0" jointxyz="0.067 -0.0275 0" jointrpy="0 0 0" />
+    <xacro:csensor plink="base_link" id="3" mass="0.001" originrpy="0 0 1.309" originxyz="-0.003 0 0" jointxyz="0.064 -0.0275 0" jointrpy="0 0 0" />
     <!-- R -->
     <xacro:csensor plink="base_link" id="4" mass="0.001" originrpy="0 0 1.0472" originxyz="-0.003 0 0" jointxyz="0.058 -0.055 0" jointrpy="0 0 0" />
     <!-- BR -->
-    <xacro:csensor plink="base_link" id="5" mass="0.001" originrpy="0 0 1.5708" originxyz="-0.003 0 0" jointxyz="-0.054 -0.035 0" jointrpy="0 0 0" />
+    <xacro:csensor plink="base_link" id="5" mass="0.001" originrpy="0 0 1.5708" originxyz="-0.003 0 0" jointxyz="-0.056 -0.035 0" jointrpy="0 0 0" />
     <!-- BL -->
-    <xacro:csensor plink="base_link" id="6" mass="0.001" originrpy="0 0 1.5708" originxyz="-0.003 0 0" jointxyz="-0.054 0.035 0" jointrpy="0 0 0" />
+    <xacro:csensor plink="base_link" id="6" mass="0.001" originrpy="0 0 1.5708" originxyz="-0.003 0 0" jointxyz="-0.056 0.035 0" jointrpy="0 0 0" />
 </robot>
